File: breakoutBoards03.kicad_pcb (KiCad board)
At the start: 2 copper layers, 100 x 100 mm, 5 parts, among them J1 CONN_24X1, J2 CONN_24X1, J3 CONN_10X1, P2 VGA, U1 48PIN

Commit message: TSOP
Parts:
- added J4: CONN_27X1, PIN_ARRAY_27X1, F.Cu at (133.0, 135.6)
- added J5: CONN_27X1, PIN_ARRAY_27X1, F.Cu at (163.5, 135.6)
- added U2: 54PIN, TSOP54_0.8mm, F.Cu at (148.3, 135.6)
- moved J3 11.0 mm to (117.8, 177.0)
- moved P2 11.0 mm to (116.5, 188.4)
Routing:
- net N-0000024: track 0.00 -> 26.5 mm
- net N-0000010: track 0.00 -> 26.5 mm
- net N-000003: track 0.00 -> 26.5 mm
- net N-0000064: track 0.00 -> 26.5 mm
- net N-0000027: track 0.00 -> 25.5 mm
- net N-000006: track 0.00 -> 25.5 mm
- net N-0000014: track 0.00 -> 25.4 mm
- net N-0000063: track 0.00 -> 25.4 mm
- net N-0000053: track 0.00 -> 23.7 mm
- net N-000008: track 0.00 -> 23.7 mm
- net N-0000042: track 0.00 -> 23.7 mm
- net N-0000056: track 0.00 -> 23.7 mm
- net N-0000012: track 0.00 -> 22.0 mm
- net N-0000048: track 0.00 -> 22.0 mm
- net N-0000049: track 0.00 -> 21.9 mm
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Other:
- board text added: "TSOP 0.8mm Breakout Board"
- board text added: "TSSOP 0.65mm Breakout Board"
- board text removed: "TSSOP Breakout Board"

Commit message: avr
Parts:
- added J6: CONN_3X1, PIN_ARRAY_3X1, F.Cu at (144.8, 196.8)
- added J7: AVRISP, AVR-ICSP, F.Cu at (144.8, 193.0)
- added J8: CONN_3X1, PIN_ARRAY_3X1, F.Cu at (144.8, 189.2)
- moved U2 2.54 mm to (150.8, 135.6)
- moved J4 2.54 mm to (135.6, 135.6)
- moved J5 2.54 mm to (166.0, 135.6)
Routing:
- net N-0000045: track 0.00 -> 2.54 mm
- net N-0000044: track 0.00 -> 2.54 mm
- net N-0000043: track 0.00 -> 2.54 mm
- net N-0000047: track 0.00 -> 2.54 mm
- net N-0000046: track 0.00 -> 2.54 mm
- net N-0000042: track 0.00 -> 2.54 mm

Commit message: soic
Parts:
- added P1: CONN_1, PIN_ARRAY_1X1, F.Cu at (154.5, 181.6)
- added P3: JTAG10, VASCH5x2, F.Cu at (166.5, 184.8)
- added P4: JTAG, VASCH10x2, F.Cu at (166.5, 195.0)
- added P5: BNC, BNC_Socket_TYCO-AMP_LargePads_RevB_20130411, F.Cu at (191.8, 108.0)
- added P6: BNCBREAKOUT, PIN_ARRAY_2X1, F.Cu at (190.5, 116.8)
- added P7: CONN_14, PIN_ARRAY_14X1, F.Cu at (197.5, 141.6)
- added P8: CONN_14, PIN_ARRAY_14X1, F.Cu at (179.1, 139.1)
- added R1: 10K, SM0805, F.Cu at (179.7, 181.9)
- added R2: 10K, SM0805, F.Cu at (179.7, 184.9)
- added R3: 10K, SM0805, F.Cu at (179.7, 187.9)
- added U3: 28PIN, SO28_BREAKOUT, F.Cu at (188.0, 140.3)
- J7: footprint AVR-ICSP -> AVR-ICSP-NOOUTLINE
- moved J6 3.86 mm to (141.0, 196.2)
- moved J7 3.86 mm to (141.0, 192.4)
- moved J8 3.86 mm to (141.0, 188.6)
Connections:
- J6 pad 1: N-0000042 (its old number) -> /AVRISPMISO
- J6 pad 2: N-0000047 (its old number) -> /AVRISPSCK
- J6 pad 3: N-0000046 (its old number) -> /AVRISPRST
- J7 pad 1: N-0000042 (its old number) -> /AVRISPMISO
- J7 pad 2: N-0000045 (its old number) -> /AVRISPVCC
- J7 pad 3: N-0000047 (its old number) -> /AVRISPSCK
- J7 pad 4: N-0000044 (its old number) -> /AVRISPMOSI
- J7 pad 5: N-0000046 (its old number) -> /AVRISPRST
- J7 pad 6: N-0000043 (its old number) -> /AVRISPGND
- J8 pad 1: N-0000045 (its old number) -> /AVRISPVCC
- J8 pad 2: N-0000044 (its old number) -> /AVRISPMOSI
- J8 pad 3: N-0000043 (its old number) -> /AVRISPGND
Routing:
- net /JTAGRESET: track 0.00 -> 23.9 mm
- net N-000004: track 0.00 -> 22.7 mm
- net /JTAGVCC: track 0.00 -> 20.8 mm
- net /JTAGTRST: track 0.00 -> 16.5 mm
- net /JTAGTCK: track 0.00 -> 15.3 mm
- net /JTAGTDI: track 0.00 -> 14.4 mm
- net /JTAGTDO: track 0.00 -> 14.3 mm
- net /JTAGTMS: track 0.00 -> 14.3 mm
- net N-0000010: track 0.00 -> 12.7 mm
- net N-0000068: track 0.00 -> 10.7 mm
- net N-0000087: track 0.00 -> 10.6 mm
- net N-0000080: track 0.00 -> 10.5 mm
- net N-0000072: track 0.00 -> 10.5 mm
- net N-0000067: track 0.00 -> 10.5 mm
- net N-0000089: track 0.00 -> 10.5 mm
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- added copper zone on B.Cu, net /BNCGND
- added copper zone on F.Cu, net /BNCGND
- added copper zone on B.Cu, net /JTAGGND
- added copper zone on F.Cu, net /JTAGGND
Other:
- net class BNC added: clearance 0.254, trace_width 1, via_dia 0.889, via_drill 0.635
- board text added: "BNC BoB"
- board text added: "BreakoutBoard03"
- board text added: "JTAG 20pin to 10pin"
- board text added: "MISO"
- board text added: "MOSI"
- board text added: "RST"
- board text added: "SCK"
- board text added: "SOIC 1.27mm Breakout Board"
- board text added: "VCC"
- board text added: "VGA Breakout Board"

Commit message: version numbers
Other:
- board text added: "BreakoutBoard03 v1"
- board text added: "https://github.com/joeferner/breakoutBoards"
- board text removed: "BreakoutBoard03"
Changed lines of the file:
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@@
     (area 99.425 80.805019 219.429002 206.169001)
     (thickness 1.6)
-    (drawings 50)
+    (drawings 51)
     (tracks 525)
     (zones 0)
@@
     )
   )
-  (gr_text BreakoutBoard03 (at 185.674 164.084) (layer F.SilkS)
+  (gr_text https://github.com/joeferner/breakoutBoards (at 170.688 175.26) (layer F.SilkS)
     (effects (font (size 1.5 1.5) (thickness 0.3)))
   )
+  (gr_text "BreakoutBoard03 v1" (at 183.896 172.466) (layer F.SilkS)
+    (effects (font (size 1.5 1.5) (thickness 0.3)))
+  )

Commit message: board 01,02,03 v1
Parts:
- added K1: CONN_3, PIN_ARRAY_3X1, F.Cu at (189.7, 165.8)
- added K2: CONN_3, PIN_ARRAY_3X1, F.Cu at (197.3, 165.8)
- added U4: 6PIN, tsot-6, F.Cu at (193.5, 165.8)
Routing:
- net N-0000099: track 0.00 -> 3.17 mm
- net N-0000094: track 0.00 -> 3.17 mm
- net N-0000097: track 0.00 -> 3.17 mm
- net N-0000095: track 0.00 -> 3.17 mm
- net N-0000098: track 0.00 -> 2.51 mm
- net N-0000096: track 0.00 -> 2.51 mm
Other:
- board text added: "TSOT-6"
