File: breakoutBoards05.kicad_pcb (KiCad board)
At the start: 2 copper layers, 16 parts, among them J1 CONN_8X1, J2 CONN_8X1, U1 MMA8453Q, U2 L3GD20

Commit message: bob 04 and 05
Parts:
- added J3: CONN_8X1, PIN_ARRAY_8X1, F.Cu at (140.5, 129.8)
- added J4: CONN_8X1, PIN_ARRAY_8X1, F.Cu at (150.6, 129.8)
- added J5: CONN_8X1, PIN_ARRAY_8X1, F.Cu at (170.7, 129.9)
- added J6: CONN_8X1, PIN_ARRAY_8X1, F.Cu at (180.8, 129.9)
- added U3: 16PIN, QFN16-0.5-3X3, F.Cu at (145.5, 131.1)
- added U4: 16PIN, LGA16-0.65-4X4, F.Cu at (175.8, 131.2)
- moved R3 17.9 mm to (180.0, 108.0)
- moved R4 12.9 mm to (177.5, 108.0)
- moved C9 10.5 mm to (165.8, 115.5), turned to 270 degrees
- moved R1 10.2 mm to (153.2, 107.8)
- moved C5 7.54 mm to (170.2, 115.5), turned to 270 degrees
- moved C6 6.96 mm to (172.8, 111.8), turned to 0 degrees
- moved C4 6.93 mm to (152.1, 110.7), turned to 0 degrees
- moved R2 5.46 mm to (151.0, 107.8)
- moved C1 5.06 mm to (147.6, 114.3), turned to 270 degrees
- moved C3 4.58 mm to (149.9, 114.3), turned to 270 degrees
- moved U2 3.48 mm to (167.8, 110.5), turned to 180 degrees
- moved U1 3.18 mm to (147.6, 109.7), turned to 180 degrees
- moved C7 3.10 mm to (168.0, 115.5), turned to 270 degrees
- moved J2 2.80 mm to (172.5, 101.6), turned to 180 degrees
- moved C2 0.57 mm to (145.5, 114.3), turned to 270 degrees
Connections:
- J1 pad 2: /ACCSCL -> /ACCINT1
- J1 pad 3: /ACCSDA -> /ACCINT2
- J1 pad 5: /ACCINT1 -> /ACCSDA
- J1 pad 6: /ACCINT2 -> /ACCSCL
Routing:
- net /ACCVDD: track 44.6 -> 32.2 mm
- net /QFN16: track 0.00 -> 9.61 mm
- net /QFN8: track 0.00 -> 9.57 mm
- net /QFN1: track 0.00 -> 9.41 mm
- net /QFN9: track 0.00 -> 9.37 mm
- net N-0000017: track 0.00 -> 8.92 mm
- net N-000008: track 0.00 -> 8.90 mm
- net N-0000015: track 0.00 -> 8.89 mm
- net N-000006: track 0.00 -> 8.89 mm
- net /GYROVDD: track 41.6 -> 49.4 mm
- net /QFN15: track 0.00 -> 7.27 mm
- net /QFN7: track 0.00 -> 7.23 mm
- net /QFN2: track 0.00 -> 7.07 mm
- net /QFN10: track 0.00 -> 7.03 mm
- net N-0000016: track 0.00 -> 6.70 mm
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Other:
- board outline added: 44 x 42.1 mm
- net class QFN added: clearance 0.2032, trace_width 0.254, via_dia 0.889, via_drill 0.635
- board text added: "LGA16-0.65-4X4 Break Out Board"
- board text added: "QFN16-0.5-3X3 Break Out Board"
