File: breakoutBoards04.kicad_pcb (KiCad board)
At the start: 2 copper layers, 39.1 x 36.6 mm, 26 parts, among them J1 USB_2, J2 CONN_10X1, M1 Mounting Hole, M2 Mounting Hole, M3 Mounting Hole, M4 Mounting Hole, U1 VREG_VOUTCENTER, U2 FT312D, X1 12MHz

Commit message: change footprint
Routing:
- net +3.3V: track 76.2 -> 80.0 mm

Commit message: bob 04 and 05
Changed lines of the file:
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@@
     (mod_text_size 1 1)
     (mod_text_width 0.15)
-    (pad_size 0.56 1.6)
+    (pad_size 0.55 1.5)
     (pad_drill 0)
     (pad_to_mask_clearance 0)
@@
     (fp_line (start 3.4 3.4) (end -3.4 3.4) (layer F.SilkS) (width 0.15))
     (fp_line (start -3.4 3.4) (end -3.4 -3.4) (layer F.SilkS) (width 0.15))
-    (pad 1 smd rect (at -2.8 4.2 270) (size 0.56 1.6)
-      (layers F.Cu F.Paste F.Mask)
-      (net 10 GND)
-    )
-    (pad 2 smd rect (at -2 4.2 270) (size 0.56 1.6)
-      (layers F.Cu F.Paste F.Mask)
-      (net 1 +3.3V)
-    )
-    (pad 3 smd rect (at -1.2 4.2 270) (size 0.56 1.6)
+    (pad 1 smd rect (at -2.8 4.2 270) (size 0.55 1.5)
+      (layers F.Cu F.Paste F.Mask)
+      (net 10 GND)
+    )
+    (pad 2 smd rect (at -2 4.2 270) (size 0.55 1.5)
+      (layers F.Cu F.Paste F.Mask)
+      (net 1 +3.3V)
+    )
+    (pad 3 smd rect (at -1.2 4.2 270) (size 0.55 1.5)
       (layers F.Cu F.Paste F.Mask)
       (net 13 N-0000011)
     )
-    (pad 4 smd rect (at -0.4 4.2 270) (size 0.56 1.6)
+    (pad 4 smd rect (at -0.4 4.2 270) (size 0.55 1.5)
       (layers F.Cu F.Paste F.Mask)
       (net 17 N-0000021)
     )
-    (pad 5 smd rect (at 0.4 4.2 270) (size 0.56 1.6)
+    (pad 5 smd rect (at 0.4 4.2 270) (size 0.55 1.5)
       (layers F.Cu F.Paste F.Mask)
       (net 18 N-0000022)
     )
-    (pad 6 smd rect (at 1.2 4.2 270) (size 0.56 1.6)
-      (layers F.Cu F.Paste F.Mask)
-      (net 10 GND)
-    )
-    (pad 7 smd rect (at 2 4.2 270) (size 0.56 1.6)
+    (pad 6 smd rect (at 1.2 4.2 270) (size 0.55 1.5)
+      (layers F.Cu F.Paste F.Mask)
+      (net 10 GND)
+    )
+    (pad 7 smd rect (at 2 4.2 270) (size 0.55 1.5)
       (layers F.Cu F.Paste F.Mask)
       (net 13 N-0000011)
     )
-    (pad 8 smd rect (at 2.8 4.2 270) (size 0.56 1.6)
-      (layers F.Cu F.Paste F.Mask)
-      (net 10 GND)
-    )
-    (pad 9 smd rect (at 4.2 2.8 270) (size 1.6 0.56)
-      (layers F.Cu F.Paste F.Mask)
-      (net 1 +3.3V)
-    )
-    (pad 10 smd rect (at 4.2 2 270) (size 1.6 0.56)
+    (pad 8 smd rect (at 2.8 4.2 270) (size 0.55 1.5)
+      (layers F.Cu F.Paste F.Mask)
+      (net 10 GND)
+    )
+    (pad 9 smd rect (at 4.2 2.8 270) (size 1.5 0.55)
+      (layers F.Cu F.Paste F.Mask)
+      (net 1 +3.3V)
+    )
+    (pad 10 smd rect (at 4.2 2 270) (size 1.5 0.55)
       (layers F.Cu F.Paste F.Mask)
       (net 4 /RESET)
     )
-    (pad 11 smd rect (at 4.2 1.2 270) (size 1.6 0.56)
+    (pad 11 smd rect (at 4.2 1.2 270) (size 1.5 0.55)
       (layers F.Cu F.Paste F.Mask)
       (net 12 N-0000010)
     )
-    (pad 12 smd rect (at 4.2 0.4 270) (size 1.6 0.56)
+    (pad 12 smd rect (at 4.2 0.4 270) (size 1.5 0.55)
       (layers F.Cu F.Paste F.Mask)
       (net 26 N-000005)
     )
-    (pad 13 smd rect (at 4.2 -0.4 270) (size 1.6 0.56)
-      (layers F.Cu F.Paste F.Mask)
-      (net 1 +3.3V)
-    )
-    (pad 14 smd rect (at 4.2 -1.2 270) (size 1.6 0.56)
-      (layers F.Cu F.Paste F.Mask)
-      (net 10 GND)
-    )
-    (pad 15 smd rect (at 4.2 -2 270) (size 1.6 0.56)
-      (layers F.Cu F.Paste F.Mask)
-      (net 10 GND)
-    )
-    (pad 16 smd rect (at 4.2 -2.8 270) (size 1.6 0.56)
-      (layers F.Cu F.Paste F.Mask)
-      (net 10 GND)
-    )
-    (pad 17 smd rect (at 2.8 -4.2 270) (size 0.56 1.6)
+    (pad 13 smd rect (at 4.2 -0.4 270) (size 1.5 0.55)
+      (layers F.Cu F.Paste F.Mask)
+      (net 1 +3.3V)
+    )
+    (pad 14 smd rect (at 4.2 -1.2 270) (size 1.5 0.55)
+      (layers F.Cu F.Paste F.Mask)
+      (net 10 GND)
+    )
+    (pad 15 smd rect (at 4.2 -2 270) (size 1.5 0.55)
+      (layers F.Cu F.Paste F.Mask)
+      (net 10 GND)
+    )
+    (pad 16 smd rect (at 4.2 -2.8 270) (size 1.5 0.55)
+      (layers F.Cu F.Paste F.Mask)
+      (net 10 GND)
+    )
+    (pad 17 smd rect (at 2.8 -4.2 270) (size 0.55 1.5)
       (layers F.Cu F.Paste F.Mask)
       (net 19 N-0000023)
     )
-    (pad 18 smd rect (at 2 -4.2 270) (size 0.56 1.6)
+    (pad 18 smd rect (at 2 -4.2 270) (size 0.55 1.5)
       (layers F.Cu F.Paste F.Mask)
       (net 22 N-0000026)
     )
-    (pad 19 smd rect (at 1.2 -4.2 270) (size 0.56 1.6)
-      (layers F.Cu F.Paste F.Mask)
-      (net 10 GND)
-    )
-    (pad 20 smd rect (at 0.4 -4.2 270) (size 0.56 1.6)
+    (pad 19 smd rect (at 1.2 -4.2 270) (size 0.55 1.5)
+      (layers F.Cu F.Paste F.Mask)
+      (net 10 GND)
+    )
+    (pad 20 smd rect (at 0.4 -4.2 270) (size 0.55 1.5)
       (layers F.Cu F.Paste F.Mask)
       (net 25 N-000004)
     )
-    (pad 21 smd rect (at -0.4 -4.2 270) (size 0.56 1.6)
+    (pad 21 smd rect (at -0.4 -4.2 270) (size 0.55 1.5)
       (layers F.Cu F.Paste F.Mask)
       (net 24 N-000003)
     )
-    (pad 22 smd rect (at -1.2 -4.2 270) (size 0.56 1.6)
-      (layers F.Cu F.Paste F.Mask)
-      (net 1 +3.3V)
-    )
-    (pad 23 smd rect (at -2 -4.2 270) (size 0.56 1.6)
+    (pad 22 smd rect (at -1.2 -4.2 270) (size 0.55 1.5)
+      (layers F.Cu F.Paste F.Mask)
+      (net 1 +3.3V)
+    )
+    (pad 23 smd rect (at -2 -4.2 270) (size 0.55 1.5)
       (layers F.Cu F.Paste F.Mask)
       (net 7 /TXD)
     )
-    (pad 24 smd rect (at -2.8 -4.2 270) (size 0.56 1.6)
+    (pad 24 smd rect (at -2.8 -4.2 270) (size 0.55 1.5)
       (layers F.Cu F.Paste F.Mask)
       (net 6 /RXD)
     )
-    (pad 25 smd rect (at -4.2 -2.8 270) (size 1.6 0.56)
+    (pad 25 smd rect (at -4.2 -2.8 270) (size 1.5 0.55)
       (layers F.Cu F.Paste F.Mask)
       (net 5 /RTS)
     )
-    (pad 26 smd rect (at -4.2 -2 270) (size 1.6 0.56)
+    (pad 26 smd rect (at -4.2 -2 270) (size 1.5 0.55)
       (layers F.Cu F.Paste F.Mask)
       (net 3 /CTS)
     )
-    (pad 27 smd rect (at -4.2 -1.2 270) (size 1.6 0.56)
-      (layers F.Cu F.Paste F.Mask)
-      (net 10 GND)
-    )
-    (pad 28 smd rect (at -4.2 -0.4 270) (size 1.6 0.56)
-      (layers F.Cu F.Paste F.Mask)
-      (net 1 +3.3V)
-    )
-    (pad 29 smd rect (at -4.2 0.4 270) (size 1.6 0.56)
+    (pad 27 smd rect (at -4.2 -1.2 270) (size 1.5 0.55)
+      (layers F.Cu F.Paste F.Mask)
+      (net 10 GND)
+    )
+    (pad 28 smd rect (at -4.2 -0.4 270) (size 1.5 0.55)
+      (layers F.Cu F.Paste F.Mask)
+      (net 1 +3.3V)
+    )
+    (pad 29 smd rect (at -4.2 0.4 270) (size 1.5 0.55)
       (layers F.Cu F.Paste F.Mask)
       (net 8 /TX_ACTIVE)
     )
-    (pad 30 smd rect (at -4.2 1.2 270) (size 1.6 0.56)
+    (pad 30 smd rect (at -4.2 1.2 270) (size 1.5 0.55)
       (layers F.Cu F.Paste F.Mask)
       (net 16 N-000002)
     )
-    (pad 31 smd rect (at -4.2 2 270) (size 1.6 0.56)
+    (pad 31 smd rect (at -4.2 2 270) (size 1.5 0.55)
       (layers F.Cu F.Paste F.Mask)
       (net 11 N-000001)
     )
-    (pad 32 smd rect (at -4.2 2.8 270) (size 1.6 0.56)
+    (pad 32 smd rect (at -4.2 2.8 270) (size 1.5 0.55)
       (layers F.Cu F.Paste F.Mask)
       (net 9 /USB_ERROR)

Commit message: added silk
Other:
- board text added: "USBERR"
Changed lines of the file:
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@@
     (area 203.118778 121.156 251.241222 160.206266)
     (thickness 1.6)
-    (drawings 48)
+    (drawings 49)
     (tracks 153)
     (zones 0)
@@
     )
   )
+  (gr_text USBERR (at 241.9 130.5 90) (layer F.SilkS)
+    (effects (font (size 0.75 0.75) (thickness 0.15)))
+  )
   (gr_text 2013-06-04 (at 219.202 152.4) (layer F.SilkS)
