File: SI4737-C40-GM/SI4737-C40-GM.kicad_pcb (KiCad board)
At the start: 2 copper layers, 19 parts, among them M1 Mounting Hole, M2 Mounting Hole, P1 AMI, P2 BREAKOUTS, P3 P03, P4 FMI, U1 SI4737-C40-GM, U2 CM1213, X1 32.768kHz

Commit message: SI4737-C40-GM-2016-05-25
Other:
- board outline added: 27 x 20.2 mm
- rule pad_to_mask_clearance: 0.2 -> 0.01
- board text added: "2016-05-25"
- board text added: "@joeferner"
- board text added: "SI4737-C40-GM Breakout Board"
Changed lines of the file:
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@@
     (links 40)
     (no_connects 0)
-    (area 0 0 0 0)
+    (area 173.124999 55.724999 200.275001 76.075001)
     (thickness 1.6)
-    (drawings 15)
+    (drawings 22)
     (tracks 155)
     (zones 0)
@@
     (pad_size 1.524 1.524)
     (pad_drill 0.762)
-    (pad_to_mask_clearance 0.2)
+    (pad_to_mask_clearance 0.01)
     (aux_axis_origin 0 0)
     (visible_elements FFFEFF7F)
     (pcbplotparams
-      (layerselection 0x00030_ffffffff)
-      (usegerberextensions false)
-      (excludeedgelayer true)
+      (layerselection 0x010f0_ffffffff)
+      (usegerberextensions true)
+      (excludeedgelayer false)
       (linewidth 0.100000)
       (plotframeref false)
@@
       (psa4output false)
       (plotreference true)
-      (plotvalue true)
+      (plotvalue false)
       (plotinvisibletext false)
       (padsonsilk false)
@@
       (outputformat 1)
       (mirror false)
-      (drillshape 1)
+      (drillshape 0)
       (scaleselection 1)
-      (outputdirectory ""))
+      (outputdirectory out/))
   )
   (net 0 "")
@@
     (pad 4 smd rect (at 1.6 -2.75 90) (size 1.9 1.3) (layers F.Cu F.Paste F.Mask))
   )
-  (module kicadlib:QFN50P300X300X60-21N (layer F.Cu)
-    (at 188.8 66.7)
-    (fp_text reference U1 (at 0 2.7) (layer F.SilkS)
-      (effects (font (size 0.6 0.6) (thickness 0.1)))
-    )
-    (fp_text value SI4737-C40-GM (at 0 0) (layer F.Fab)
-      (effects (font (size 0.6 0.6) (thickness 0.1)))
-    )
-    (fp_line (start -2.15 2.15) (end -2.15 -2.15) (layer F.CrtYd) (width 0.15))
-    (fp_line (start 2.15 2.15) (end -2.15 2.15) (layer F.CrtYd) (width 0.15))
-    (fp_line (start 2.15 -2.15) (end 2.15 2.15) (layer F.CrtYd) (width 0.15))
-    (fp_line (start -2.15 -2.15) (end 2.15 -2.15) (layer F.CrtYd) (width 0.15))
-    (fp_line (start -1.5 1.5) (end -1.5 -1.5) (layer F.SilkS) (width 0.15))
-    (fp_line (start 1.5 1.5) (end -1.5 1.5) (layer F.SilkS) (width 0.15))
-    (fp_line (start 1.5 -1.5) (end 1.5 1.5) (layer F.SilkS) (width 0.15))
-    (fp_line (start -1.5 -1.5) (end 1.5 -1.5) (layer F.SilkS) (width 0.15))
-    (pad 2 smd rect (at -1.75 -0.75) (size 1.3 0.3) (layers F.Cu F.Paste F.Mask)
-      (net 10 /FMI))
-    (pad 3 smd rect (at -1.75 -0.25) (size 1.3 0.3) (layers F.Cu F.Paste F.Mask)
-      (net 1 GNDPWR))
-    (pad 4 smd rect (at -1.75 0.25) (size 1.3 0.3) (layers F.Cu F.Paste F.Mask)
-      (net 12 /AMI))
-    (pad 5 smd rect (at -1.75 0.75) (size 1.3 0.3) (layers F.Cu F.Paste F.Mask)
-      (net 11 /RST))
-    (pad 1 smd rect (at -1.75 -1.75) (size 1.3 1.3) (layers F.Cu F.Paste F.Mask)
-      (net 13 "Net-(U1-Pad1)"))
-    (pad 6 smd rect (at -1.75 1.75) (size 1.3 1.3) (layers F.Cu F.Paste F.Mask)
-      (net 14 /SEN))
-    (pad 7 smd rect (at -0.75 1.75) (size 0.3 1.3) (layers F.Cu F.Paste F.Mask)
-      (net 15 /SCLK))
-    (pad 8 smd rect (at -0.25 1.75) (size 0.3 1.3) (layers F.Cu F.Paste F.Mask)
-      (net 16 /SDIO))
-    (pad 9 smd rect (at 0.25 1.75) (size 0.3 1.3) (layers F.Cu F.Paste F.Mask)
-      (net 3 "Net-(C2-Pad1)"))
-    (pad 10 smd rect (at 0.75 1.75) (size 0.3 1.3) (layers F.Cu F.Paste F.Mask)
-      (net 2 +3.3V))
-    (pad 11 smd rect (at 1.75 1.75) (size 1.3 1.3) (layers F.Cu F.Paste F.Mask)
-      (net 2 +3.3V))
-    (pad 12 smd rect (at 1.75 0.75) (size 1.3 0.3) (layers F.Cu F.Paste F.Mask)
-      (net 1 GNDPWR))
-    (pad 13 smd rect (at 1.75 0.25) (size 1.3 0.3) (layers F.Cu F.Paste F.Mask)
-      (net 6 "Net-(C5-Pad2)"))
-    (pad 14 smd rect (at 1.75 -0.25) (size 1.3 0.3) (layers F.Cu F.Paste F.Mask)
-      (net 8 "Net-(C6-Pad2)"))
-    (pad 15 smd rect (at 1.75 -0.75) (size 1.3 0.3) (layers F.Cu F.Paste F.Mask)
-      (net 17 /DOUT))
-    (pad 16 smd rect (at 1.75 -1.75) (size 1.3 1.3) (layers F.Cu F.Paste F.Mask)
-      (net 18 /DFS))
-    (pad 17 smd rect (at 0.75 -1.75) (size 0.3 1.3) (layers F.Cu F.Paste F.Mask)
-      (net 4 "Net-(C3-Pad1)"))
-    (pad 18 smd rect (at 0.25 -1.75) (size 0.3 1.3) (layers F.Cu F.Paste F.Mask)
-      (net 21 /GPO2))
-    (pad 19 smd rect (at -0.25 -1.75) (size 0.3 1.3) (layers F.Cu F.Paste F.Mask)
-      (net 19 /GPO1))
-    (pad 20 smd rect (at -0.75 -1.75) (size 0.3 1.3) (layers F.Cu F.Paste F.Mask)
-      (net 20 "Net-(U1-Pad20)"))
-    (pad 21 smd rect (at 0 0) (size 1.75 1.75) (layers F.Cu F.Paste F.Mask)
-      (net 1 GNDPWR))
-  )
   (module kicadlib:MTGNP565H328Z565P (layer F.Cu)
     (at 176.7 59.2)
@@
       (net 1 GNDPWR))
   )
+  (module kicadlib:QFN50P300X300X60-21N (layer F.Cu)
+    (at 188.8 66.7)
+    (fp_text reference U1 (at 0 2.9) (layer F.SilkS)
+      (effects (font (size 0.6 0.6) (thickness 0.1)))
+    )
+    (fp_text value SI4737-C40-GM (at 0 0) (layer F.Fab)
+      (effects (font (size 0.6 0.6) (thickness 0.1)))
+    )
+    (fp_circle (center -2.921 -2.794) (end -2.794 -2.667) (layer F.SilkS) (width 0.3))
+    (fp_line (start -2.15 2.15) (end -2.15 -2.15) (layer F.CrtYd) (width 0.15))
+    (fp_line (start 2.15 2.15) (end -2.15 2.15) (layer F.CrtYd) (width 0.15))
+    (fp_line (start 2.15 -2.15) (end 2.15 2.15) (layer F.CrtYd) (width 0.15))
+    (fp_line (start -2.15 -2.15) (end 2.15 -2.15) (layer F.CrtYd) (width 0.15))
+    (fp_line (start -1.5 1.5) (end -1.5 -1.5) (layer F.SilkS) (width 0.15))
+    (fp_line (start 1.5 1.5) (end -1.5 1.5) (layer F.SilkS) (width 0.15))
+    (fp_line (start 1.5 -1.5) (end 1.5 1.5) (layer F.SilkS) (width 0.15))
+    (fp_line (start -1.5 -1.5) (end 1.5 -1.5) (layer F.SilkS) (width 0.15))
+    (pad 2 smd rect (at -1.75 -0.75) (size 1.3 0.3) (layers F.Cu F.Paste F.Mask)
+      (net 10 /FMI))
+    (pad 3 smd rect (at -1.75 -0.25) (size 1.3 0.3) (layers F.Cu F.Paste F.Mask)
+      (net 1 GNDPWR))
+    (pad 4 smd rect (at -1.75 0.25) (size 1.3 0.3) (layers F.Cu F.Paste F.Mask)
+      (net 12 /AMI))
+    (pad 5 smd rect (at -1.75 0.75) (size 1.3 0.3) (layers F.Cu F.Paste F.Mask)
+      (net 11 /RST))
+    (pad 1 smd rect (at -1.75 -1.75) (size 1.3 1.3) (layers F.Cu F.Paste F.Mask)
+      (net 13 "Net-(U1-Pad1)"))
+    (pad 6 smd rect (at -1.75 1.75) (size 1.3 1.3) (layers F.Cu F.Paste F.Mask)
+      (net 14 /SEN))
+    (pad 7 smd rect (at -0.75 1.75) (size 0.3 1.3) (layers F.Cu F.Paste F.Mask)
+      (net 15 /SCLK))
+    (pad 8 smd rect (at -0.25 1.75) (size 0.3 1.3) (layers F.Cu F.Paste F.Mask)
+      (net 16 /SDIO))
+    (pad 9 smd rect (at 0.25 1.75) (size 0.3 1.3) (layers F.Cu F.Paste F.Mask)
+      (net 3 "Net-(C2-Pad1)"))
+    (pad 10 smd rect (at 0.75 1.75) (size 0.3 1.3) (layers F.Cu F.Paste F.Mask)
+      (net 2 +3.3V))
+    (pad 11 smd rect (at 1.75 1.75) (size 1.3 1.3) (layers F.Cu F.Paste F.Mask)
+      (net 2 +3.3V))
+    (pad 12 smd rect (at 1.75 0.75) (size 1.3 0.3) (layers F.Cu F.Paste F.Mask)
+      (net 1 GNDPWR))
+    (pad 13 smd rect (at 1.75 0.25) (size 1.3 0.3) (layers F.Cu F.Paste F.Mask)
+      (net 6 "Net-(C5-Pad2)"))
+    (pad 14 smd rect (at 1.75 -0.25) (size 1.3 0.3) (layers F.Cu F.Paste F.Mask)
+      (net 8 "Net-(C6-Pad2)"))
+    (pad 15 smd rect (at 1.75 -0.75) (size 1.3 0.3) (layers F.Cu F.Paste F.Mask)
+      (net 17 /DOUT))
+    (pad 16 smd rect (at 1.75 -1.75) (size 1.3 1.3) (layers F.Cu F.Paste F.Mask)
+      (net 18 /DFS))
+    (pad 17 smd rect (at 0.75 -1.75) (size 0.3 1.3) (layers F.Cu F.Paste F.Mask)
+      (net 4 "Net-(C3-Pad1)"))
+    (pad 18 smd rect (at 0.25 -1.75) (size 0.3 1.3) (layers F.Cu F.Paste F.Mask)
+      (net 21 /GPO2))
+    (pad 19 smd rect (at -0.25 -1.75) (size 0.3 1.3) (layers F.Cu F.Paste F.Mask)
+      (net 19 /GPO1))
+    (pad 20 smd rect (at -0.75 -1.75) (size 0.3 1.3) (layers F.Cu F.Paste F.Mask)
+      (net 20 "Net-(U1-Pad20)"))
+    (pad 21 smd rect (at 0 0) (size 1.75 1.75) (layers F.Cu F.Paste F.Mask)
+      (net 1 GNDPWR))
+  )
+  (gr_text @joeferner (at 186.9 58.9) (layer B.SilkS)
+    (effects (font (size 0.6 0.6) (thickness 0.1)) (justify mirror))
+  )
+  (gr_text 2016-05-25 (at 186.9 57.8) (layer B.SilkS)
+    (effects (font (size 0.6 0.6) (thickness 0.1)) (justify mirror))
+  )
+  (gr_text "SI4737-C40-GM Breakout Board" (at 186.9 56.8) (layer B.SilkS)
+    (effects (font (size 0.6 0.6) (thickness 0.1)) (justify mirror))
+  )
+  (gr_line (start 173.2 76) (end 173.2 55.8) (layer Edge.Cuts) (width 0.15))
+  (gr_line (start 200.2 76) (end 173.2 76) (layer Edge.Cuts) (width 0.15))
+  (gr_line (start 200.2 55.8) (end 200.2 76) (layer Edge.Cuts) (width 0.15))
+  (gr_line (start 173.2 55.8) (end 200.2 55.8) (layer Edge.Cuts) (width 0.15))
   (gr_text FMI (at 180 63.5) (layer F.SilkS)
     (effects (font (size 0.6 0.6) (thickness 0.1)))
